File: .history/Keyboard_USB_Adapter.kicad_sch (KiCad schematic)
At the start: 9 parts, among them J1 USB_C_Receptacle_USB2.0_16P, J2 Conn_01x05, SW1 SW_SPDT, U1 USBLC6-2SC6

Commit message: placed parts
Connections:
- net GND: now reaches J1.A1 (GND), J1.A12 (GND), J1.B1 (GND), J1.B12 (GND)
- net GND: now also J1.SH (SHIELD)
- net VBUS: now reaches J1.A4 (VBUS), J1.A9 (VBUS), J1.B4 (VBUS), J1.B9 (VBUS)
- net VBUS: now also F1.2
- net at J1.A6 (D+): now also J1.B6 (D+)
- net at J1.A7 (D-): now also J1.B7 (D-)
Other:
- moved on the sheet: C1, C2, J2, R1, R2, U1

Commit message: Progress
Parts:
- C1: value C -> 10nF
- C2: value C -> 100nF
- F1: value Polyfuse -> 500mA
- R1, R2: value R -> 5.1K
Connections:
- net GND: now also R1.1, R2.1
- net VBUS: no longer F1.2
- net at J1.A5 (CC1): now also R2.2
- net at J1.B5 (CC2): now also R1.2
Other:
- moved on the sheet: C1, C2, J1, J2, R1, R2, SW1, U1

Commit message: finished switch
Connections:
- net GND: now also U1.1 (I/O1)
- net VBUS: now also F1.1
Other:
- moved on the sheet: J2, SW1, U1
Changed lines of the file:
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@@
+	(wire
+		(pts
+			(xy 60.96 113.03) (xy 60.96 118.11)
+		)
+		(stroke
+			(width 0)
+			(type default)
+		)
+	)
 	(wire
 		(pts
@@
 	(wire
 		(pts
-			(xy 57.15 93.98) (xy 57.15 96.52)
+			(xy 68.58 113.03) (xy 60.96 113.03)
 		)
 		(stroke
@@
 	(wire
 		(pts
-			(xy 76.2 83.82) (xy 76.2 87.63)
+			(xy 57.15 93.98) (xy 57.15 96.52)
 		)
 		(stroke
@@
 		)
 	)
+	(wire
+		(pts
+			(xy 76.2 83.82) (xy 76.2 87.63)
+		)
+		(stroke
+			(width 0)
+			(type default)
+		)
+	)
 	(symbol
 		(lib_id "Connector:USB_C_Receptacle_USB2.0_16P")
@@
 	(symbol
 		(lib_id "Switch:SW_SPDT")
-		(at 86.36 120.65 0)
+		(at 113.03 121.92 0)
 		(unit 1)
 		(body_style 1)
@@
 		(fields_autoplaced yes)
 		(property "Reference" "SW1"
-			(at 86.36 111.76 0)
+			(at 113.03 113.03 0)
 			(show_name no)
 			(do_not_autoplace no)
@@
 		)
 		(property "Value" "SW_SPDT"
-			(at 86.36 114.3 0)
-			(show_name no)
-			(do_not_autoplace no)
-			(effects
-				(font
-					(size 1.27 1.27)
-				)
-			)
-		)
-		(property "Footprint" ""
-			(at 86.36 120.65 0)
+			(at 113.03 115.57 0)
+			(show_name no)
+			(do_not_autoplace no)
+			(effects
+				(font
+					(size 1.27 1.27)
+				)
+			)
+		)
+		(property "Footprint" ""
+			(at 113.03 121.92 0)
 			(hide yes)
 			(show_name no)
@@
 		)
 		(property "Datasheet" ""
-			(at 86.36 128.27 0)
+			(at 113.03 129.54 0)
 			(hide yes)
 			(show_name no)
@@
 		)
 		(property "Description" "Switch, single pole double throw"
-			(at 86.36 120.65 0)
+			(at 113.03 121.92 0)
 			(hide yes)
 			(show_name no)
@@
 				(path "/5abeb7b7-6d19-4686-bb3f-ba353c7d837b"
 					(reference "SW1")
+					(unit 1)
+				)
+			)
+		)
+	)
+	(symbol
+		(lib_id "power:VBUS")
+		(at 67.31 60.96 0)
+		(unit 1)
+		(body_style 1)
+		(exclude_from_sim no)
+		(in_bom yes)
+		(on_board yes)
+		(in_pos_files yes)
+		(dnp no)
+		(fields_autoplaced yes)
+		(property "Reference" "#PWR07"
+			(at 67.31 64.77 0)
+			(hide yes)
+			(show_name no)
+			(do_not_autoplace no)
+			(effects
+				(font
+					(size 1.27 1.27)
+				)
+			)
+		)
+		(property "Value" "VBUS"
+			(at 67.31 55.88 0)
+			(show_name no)
+			(do_not_autoplace no)
+			(effects
+				(font
+					(size 1.27 1.27)
+				)
+			)
+		)
+		(property "Footprint" ""
+			(at 67.31 60.96 0)
+			(hide yes)
+			(show_name no)
+			(do_not_autoplace no)
+			(effects
+				(font
+					(size 1.27 1.27)
+				)
+			)
+		)
+		(property "Datasheet" ""
+			(at 67.31 60.96 0)
+			(hide yes)
+			(show_name no)
+			(do_not_autoplace no)
+			(effects
+				(font
+					(size 1.27 1.27)
+				)
+			)
+		)
+		(property "Description" "Power symbol creates a global label with name \"VBUS\""
+			(at 67.31 60.96 0)
+			(hide yes)
+			(show_name no)
+			(do_not_autoplace no)
+			(effects
+				(font
+					(size 1.27 1.27)
+				)
+			)
+		)
+		(pin "1"
+		)
+		(instances
+			(project "Keyboard_USB_Adapter"
+				(path "/5abeb7b7-6d19-4686-bb3f-ba353c7d837b"
+					(reference "#PWR07")
 					(unit 1)
 				)
@@
 	(symbol
 		(lib_id "Power_Protection:USBLC6-2SC6")
-		(at 90.17 54.61 0)
+		(at 73.66 113.03 0)
 		(unit 1)
 		(body_style 1)
@@
 		(fields_autoplaced yes)
 		(property "Reference" "U1"
-			(at 91.8211 46.99 0)
+			(at 75.3111 105.41 0)
 			(show_name no)
 			(do_not_autoplace no)
@@
 		)
 		(property "Value" "USBLC6-2SC6"
-			(at 91.8211 49.53 0)
+			(at 75.3111 107.95 0)
 			(show_name no)
 			(do_not_autoplace no)
@@
 		)
 		(property "Footprint" "Package_TO_SOT_SMD:SOT-23-6"
-			(at 91.44 60.96 0)
+			(at 74.93 119.38 0)
 			(hide yes)
 			(show_name no)
@@
 		)
 		(property "Datasheet" "https://www.st.com/resource/en/datasheet/usblc6-2.pdf"
-			(at 91.44 62.865 0)
+			(at 74.93 121.285 0)
 			(hide yes)
 			(show_name no)
@@
 		)
 		(property "Description" "Very low capacitance ESD protection diode, 2 data-line, SOT-23-6"
-			(at 90.17 54.61 0)
+			(at 73.66 113.03 0)
 			(hide yes)
 			(show_name no)
@@
 	(symbol
 		(lib_id "Connector_Generic:Conn_01x05")
-		(at 100.33 109.22 0)
+		(at 111.76 102.87 0)
 		(unit 1)
 		(body_style 1)
@@
 		(fields_autoplaced yes)
 		(property "Reference" "J2"
-			(at 102.87 107.9499 0)
+			(at 114.3 101.5999 0)
 			(show_name no)
 			(do_not_autoplace no)
@@
 		)
 		(property "Value" "Conn_01x05"
-			(at 102.87 110.4899 0)
+			(at 114.3 104.1399 0)
 			(show_name no)
 			(do_not_autoplace no)
@@
 		)
 		(property "Footprint" ""
-			(at 100.33 109.22 0)
+			(at 111.76 102.87 0)
 			(hide yes)
 			(show_name no)
@@
 		)
 		(property "Datasheet" ""
-			(at 100.33 109.22 0)
+			(at 111.76 102.87 0)
 			(hide yes)
 			(show_name no)
@@
 		)
 		(property "Description" "Generic connector, single row, 01x05, script generated (kicad-library-utils/schlib/autogen/connector/)"
-			(at 100.33 109.22 0)
+			(at 111.76 102.87 0)
 			(hide yes)
 			(show_name no)
@@
 					(unit 1)
 				)
+			)
+		)
+	)
+	(symbol
+		(lib_id "power:GND")
+		(at 60.96 118.11 0)
+		(unit 1)
+		(body_style 1)
+		(exclude_from_sim no)
+		(in_bom yes)
+		(on_board yes)
+		(in_pos_files yes)
+		(dnp no)
+		(fields_autoplaced yes)
+		(property "Reference" "#PWR06"
+			(at 60.96 124.46 0)
+			(hide yes)
+			(show_name no)
+			(do_not_autoplace no)
+			(effects
+				(font
+					(size 1.27 1.27)
+				)
+			)
+		)
+		(property "Value" "GND"
+			(at 60.96 123.19 0)
+			(show_name no)
+			(do_not_autoplace no)
+			(effects
+				(font
+					(size 1.27 1.27)
+				)
+			)
+		)
+		(property "Footprint" ""
+			(at 60.96 118.11 0)
+			(hide yes)
+			(show_name no)
+			(do_not_autoplace no)
+			(effects
+				(font
+					(size 1.27 1.27)
+				)
+			)
+		)
+		(property "Datasheet" ""
+			(at 60.96 118.11 0)
+			(hide yes)
+			(show_name no)
+			(do_not_autoplace no)
+			(effects
+				(font
+					(size 1.27 1.27)
+				)
+			)
+		)
+		(property "Description" "Power symbol creates a global label with name \"GND\" , ground"
+			(at 60.96 118.11 0)
+			(hide yes)
+			(show_name no)
+			(do_not_autoplace no)
+			(effects
+				(font
+					(size 1.27 1.27)
+				)
+			)
+		)
+		(pin "1"
+		)
+		(instances
+			(project "Keyboard_USB_Adapter"
+				(path "/5abeb7b7-6d19-4686-bb3f-ba353c7d837b"
+					(reference "#PWR06")
+					(unit 1)
+				)
